File: hardware/CarteAlim/carteAlim.brd (EAGLE design)
At the start: 30.5 x 99.1 mm, 19 parts

Commit message: Voilà le patch de la carte d'alim!
Parts:
- removed C1, C3, C5: (no value), resistor:E2-5
- removed C2, C4, C6: (no value), resistor:E2,5-6
- removed L1, L2, L3: (no value), inductor-neosid:SD12K100
- moved DC1 38.3 mm to (24.1, 48.3)
- moved DC2 30.7 mm to (24.1, 31.8)
Connections:
- removed net N$3: C2.+, DC1.1, L1.2
- removed net N$4: C4.+, DC2.1, L2.2
- removed net N$7: C1.+, C3.+, C5.+, L1.1, L2.1, L3.1, X4.1
- removed net N$8: C6.+, DC3.1, L3.2
- new net ALIM-SSC: DC1.1, DC2.1, DC3.1, X4.1, X6.1
- net +5V-ALIM-SSC-RASP: no longer X6.1
- net GND: no longer C1.-, C2.-, C3.-, C4.-, C5.-, C6.-
Routing:
- net N$7: track 104.3 -> 0.00 mm
- net ALIM-SSC: track 0.00 -> 89.2 mm
- net N$5: track 14.5 -> 54.9 mm
- net N$6: track 24.0 -> 59.2 mm
- net N$8: track 17.8 -> 0.00 mm
- net N$3: track 15.8 -> 0.00 mm
- net N$4: track 15.5 -> 0.00 mm
- net +5V-ALIM-SSC-RASP: track 63.7 -> 48.9 mm
