File: hardware/CarteAlim/carteAlim.sch (EAGLE design)
At the start: 19 parts

Commit message: Voilà le patch de la carte d'alim!
Parts:
- removed C1, C3, C5: (no value), resistor:CPOL-USE2-5
- removed C2, C4, C6: (no value), resistor:CPOL-USE2.5-6
- removed L1, L2, L3: (no value), inductor-neosid:SD12K100
Connections:
- removed net N$3: C2.+, DC1.VIN, L1.2
- removed net N$4: C4.+, DC2.VIN, L2.2
- removed net N$7: C1.+, C3.+, C5.+, L1.1, L2.1, L3.1, X4-1.KL
- removed net N$8: C6.+, DC3.VIN, L3.2
- new net ALIM-SSC: DC1.VIN, DC2.VIN, DC3.VIN, X4-1.KL, X6-1.KL
- net +5V-ALIM-SSC-RASP: no longer X6-1.KL
- net GND: no longer C1.-, C2.-, C3.-, C4.-, C5.-, C6.-
Changed lines of the file:
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@@
 <?xml version="1.0" encoding="utf-8"?>
 <!DOCTYPE eagle SYSTEM "eagle.dtd">
-<eagle version="6.3">
+<eagle version="6.4">
 <drawing>
 <settings>
@@
 <part name="SUPPLY5" library="supply2" deviceset="GND" device=""/>
 <part name="SUPPLY6" library="supply2" deviceset="GND" device=""/>
-<part name="L1" library="inductor-neosid" deviceset="SD12" device="K100"/>
-<part name="L2" library="inductor-neosid" deviceset="SD12" device="K100"/>
-<part name="L3" library="inductor-neosid" deviceset="SD12" device="K100"/>
-<part name="C1" library="resistor" deviceset="CPOL-US" device="E2-5"/>
-<part name="C2" library="resistor" deviceset="CPOL-US" device="E2.5-6"/>
-<part name="C3" library="resistor" deviceset="CPOL-US" device="E2-5"/>
-<part name="C4" library="resistor" deviceset="CPOL-US" device="E2.5-6"/>
-<part name="C5" library="resistor" deviceset="CPOL-US" device="E2-5"/>
-<part name="C6" library="resistor" deviceset="CPOL-US" device="E2.5-6"/>
 <part name="X6" library="con-ptr500" deviceset="AK300/2" device=""/>
 <part name="SUPPLY7" library="supply2" deviceset="GND" device=""/>
@@
 <instance part="SUPPLY5" gate="GND" x="106.68" y="30.48"/>
 <instance part="SUPPLY6" gate="GND" x="106.68" y="63.5"/>
-<instance part="L1" gate="G$1" x="45.72" y="73.66"/>
-<instance part="L2" gate="G$1" x="45.72" y="40.64"/>
-<instance part="L3" gate="G$1" x="45.72" y="7.62"/>
-<instance part="C1" gate="G$1" x="33.02" y="71.12"/>
-<instance part="C2" gate="G$1" x="55.88" y="71.12"/>
-<instance part="C3" gate="G$1" x="33.02" y="38.1"/>
-<instance part="C4" gate="G$1" x="55.88" y="38.1"/>
-<instance part="C5" gate="G$1" x="33.02" y="5.08"/>
-<instance part="C6" gate="G$1" x="55.88" y="5.08"/>
 <instance part="X6" gate="-1" x="96.52" y="-15.24"/>
 <instance part="X6" gate="-2" x="96.52" y="-20.32"/>
@@
 </segment>
 <segment>
-<pinref part="X6" gate="-1" pin="KL"/>
-<wire x1="101.6" y1="-15.24" x2="104.14" y2="-15.24" width="0.1524" layer="91"/>
-<wire x1="104.14" y1="-15.24" x2="104.14" y2="-12.7" width="0.1524" layer="91"/>
-<label x="104.14" y="-12.7" size="1.778" layer="95" xref="yes"/>
-</segment>
-<segment>
 <pinref part="SV1" gate="G$1" pin="1"/>
 <pinref part="SV1" gate="G$1" pin="9"/>
@@
 </segment>
 </net>
-<net name="N$7" class="0">
+<net name="ALIM-SSC" class="0">
 <segment>
 <wire x1="25.4" y1="73.66" x2="25.4" y2="40.64" width="0.1524" layer="91"/>
@@
 <pinref part="X4" gate="-1" pin="KL"/>
 <wire x1="25.4" y1="40.64" x2="25.4" y2="7.62" width="0.1524" layer="91"/>
-<pinref part="L1" gate="G$1" pin="1"/>
-<wire x1="25.4" y1="73.66" x2="33.02" y2="73.66" width="0.1524" layer="91"/>
-<pinref part="L2" gate="G$1" pin="1"/>
-<wire x1="33.02" y1="73.66" x2="40.64" y2="73.66" width="0.1524" layer="91"/>
-<wire x1="40.64" y1="40.64" x2="33.02" y2="40.64" width="0.1524" layer="91"/>
-<pinref part="L3" gate="G$1" pin="1"/>
-<wire x1="33.02" y1="40.64" x2="25.4" y2="40.64" width="0.1524" layer="91"/>
-<wire x1="25.4" y1="7.62" x2="33.02" y2="7.62" width="0.1524" layer="91"/>
-<pinref part="C1" gate="G$1" pin="+"/>
-<junction x="33.02" y="73.66"/>
-<pinref part="C3" gate="G$1" pin="+"/>
-<junction x="33.02" y="40.64"/>
-<pinref part="C5" gate="G$1" pin="+"/>
-<wire x1="33.02" y1="7.62" x2="40.64" y2="7.62" width="0.1524" layer="91"/>
-<junction x="33.02" y="7.62"/>
+<wire x1="25.4" y1="73.66" x2="60.96" y2="73.66" width="0.1524" layer="91"/>
+<wire x1="60.96" y1="40.64" x2="25.4" y2="40.64" width="0.1524" layer="91"/>
+<wire x1="25.4" y1="7.62" x2="50.8" y2="7.62" width="0.1524" layer="91"/>
+<pinref part="DC1" gate="G$1" pin="VIN"/>
+<pinref part="DC2" gate="G$1" pin="VIN"/>
+<pinref part="DC3" gate="G$1" pin="VIN"/>
+<wire x1="50.8" y1="7.62" x2="53.34" y2="7.62" width="0.1524" layer="91"/>
+<wire x1="53.34" y1="7.62" x2="60.96" y2="7.62" width="0.1524" layer="91"/>
+<label x="25.4" y="7.62" size="1.778" layer="95" rot="R270" xref="yes"/>
+</segment>
+<segment>
+<pinref part="X6" gate="-1" pin="KL"/>
+<wire x1="101.6" y1="-15.24" x2="104.14" y2="-15.24" width="0.1524" layer="91"/>
+<wire x1="104.14" y1="-15.24" x2="104.14" y2="-12.7" width="0.1524" layer="91"/>
+<label x="104.14" y="-12.7" size="1.778" layer="95" xref="yes"/>
 </segment>
 </net>
@@
 <wire x1="73.66" y1="66.04" x2="73.66" y2="63.5" width="0.1524" layer="91"/>
 <pinref part="SUPPLY1" gate="GND" pin="GND"/>
-<wire x1="73.66" y1="63.5" x2="55.88" y2="63.5" width="0.1524" layer="91"/>
-<pinref part="C1" gate="G$1" pin="-"/>
-<wire x1="55.88" y1="63.5" x2="33.02" y2="63.5" width="0.1524" layer="91"/>
-<wire x1="33.02" y1="66.04" x2="33.02" y2="63.5" width="0.1524" layer="91"/>
-<pinref part="C2" gate="G$1" pin="-"/>
-<wire x1="55.88" y1="66.04" x2="55.88" y2="63.5" width="0.1524" layer="91"/>
 </segment>
 <segment>
@@
 <wire x1="73.66" y1="33.02" x2="73.66" y2="30.48" width="0.1524" layer="91"/>
 <pinref part="SUPPLY2" gate="GND" pin="GND"/>
-<wire x1="73.66" y1="30.48" x2="55.88" y2="30.48" width="0.1524" layer="91"/>
-<pinref part="C3" gate="G$1" pin="-"/>
-<wire x1="55.88" y1="30.48" x2="33.02" y2="30.48" width="0.1524" layer="91"/>
-<wire x1="33.02" y1="33.02" x2="33.02" y2="30.48" width="0.1524" layer="91"/>
-<pinref part="C4" gate="G$1" pin="-"/>
-<wire x1="55.88" y1="33.02" x2="55.88" y2="30.48" width="0.1524" layer="91"/>
 </segment>
 <segment>
@@
 <junction x="88.9" y="0"/>
 <wire x1="88.9" y1="0" x2="101.6" y2="0" width="0.1524" layer="91"/>
-<wire x1="73.66" y1="0" x2="55.88" y2="0" width="0.1524" layer="91"/>
-<pinref part="C5" gate="G$1" pin="-"/>
-<wire x1="55.88" y1="0" x2="33.02" y2="0" width="0.1524" layer="91"/>
-<pinref part="C6" gate="G$1" pin="-"/>
-<junction x="55.88" y="0"/>
 </segment>
 <segment>
@@
 </segment>
 </net>
-<net name="N$3" class="0">
-<segment>
-<pinref part="L1" gate="G$1" pin="2"/>
-<pinref part="DC1" gate="G$1" pin="VIN"/>
-<wire x1="50.8" y1="73.66" x2="55.88" y2="73.66" width="0.1524" layer="91"/>
-<pinref part="C2" gate="G$1" pin="+"/>
-<wire x1="55.88" y1="73.66" x2="60.96" y2="73.66" width="0.1524" layer="91"/>
-<junction x="55.88" y="73.66"/>
-</segment>
-</net>
-<net name="N$4" class="0">
-<segment>
-<pinref part="DC2" gate="G$1" pin="VIN"/>
-<pinref part="L2" gate="G$1" pin="2"/>
-<wire x1="60.96" y1="40.64" x2="55.88" y2="40.64" width="0.1524" layer="91"/>
-<pinref part="C4" gate="G$1" pin="+"/>
-<wire x1="55.88" y1="40.64" x2="50.8" y2="40.64" width="0.1524" layer="91"/>
-<junction x="55.88" y="40.64"/>
-</segment>
-</net>
-<net name="N$8" class="0">
-<segment>
-<pinref part="L3" gate="G$1" pin="2"/>
-<pinref part="DC3" gate="G$1" pin="VIN"/>
-<wire x1="50.8" y1="7.62" x2="55.88" y2="7.62" width="0.1524" layer="91"/>
-<pinref part="C6" gate="G$1" pin="+"/>
-<wire x1="55.88" y1="7.62" x2="60.96" y2="7.62" width="0.1524" layer="91"/>
-<junction x="55.88" y="7.62"/>
-</segment>
-</net>
